File: hw/kicad_v1_1/projects/control_board/mcu_rtc.sch (KiCad schematic (older format))
At the start: 9 parts, among them U2 MCP7940N, Y1 32.768kHz

Commit message: Update
Begin work on updating for rev1.1.
Connections:
- net labels added: +5V
- net labels removed: +3.3V
Changed lines of the file:
@@
-	1    0    0    -1
-$EndComp
-$Comp
-L +3.3V #PWR036
-U 1 1 575E35A4
-P 6600 2700
-F 0 "#PWR036" H 6600 2550 50  0001 C CNN
-F 1 "+3.3V" H 6600 2840 50  0000 C CNN
-F 2 "" H 6600 2700 50  0000 C CNN
-F 3 "" H 6600 2700 50  0000 C CNN
-	1    6600 2700
 	1    0    0    -1
 $EndComp
@@
 	4400 4600 3250 4600
 Connection ~ 3250 4600
+$Comp
+L +5V #PWR?
+U 1 1 581F2E8E
+P 6600 2700
+F 0 "#PWR?" H 6600 2550 50  0001 C CNN
+F 1 "+5V" H 6600 2840 50  0000 C CNN
+F 2 "" H 6600 2700 50  0000 C CNN
+F 3 "" H 6600 2700 50  0000 C CNN
+	1    6600 2700
+	1    0    0    -1
+$EndComp
 $EndSCHEMATC
