File: hw/kicad_v1_1/projects/control_board/nixie_power_supply.sch (KiCad schematic (older format))
At the start: 22 parts, among them Q1 IPB50R199CP, U1 MAX1771

Commit message: Schematic Work Complete
Check in schematic work before touching PCB. This should give me a point
to go back to if it all goes to hell.
Parts:
- removed Q? (x2): MPSA42, TO-92, symbol MPSA42
- added C?: 100uF, Capacitors_Tantalum_SMD:TantalC_SizeD_EIA-7343_HandSoldering, symbol C-RESCUE-nixie_clock
- added Q? (x2): MMBTA42, TO_SOT_Packages_SMD:SOT-23_Handsoldering, symbol MMBTA42
- added R?: 5K, symbol RVAR
- L1: value 150u -> 100u
- R3: value 0.1 -> 0.05
- R4: value 1.123MEG -> 1.5MEG
Connections:
- net labels added: +180V, 180V_EN
- net labels removed: +170V, 180V_SHDN
- wire segments 54 -> 58
Other:
- note added: ">2A max current"
- moved on the sheet: R2
Changed lines of the file:
@@
 P 6000 5600
 F 0 "R3" V 6080 5600 40  0000 C CNN
-F 1 "0.1" V 6007 5601 40  0000 C CNN
+F 1 "0.05" V 6007 5601 40  0000 C CNN
 F 2 "Resistors_SMD:R_0805_HandSoldering" V 5930 5600 30  0001 C CNN
 F 3 "~" H 6000 5600 30  0000 C CNN
@@
 L R-RESCUE-nixie_clock R2
 U 1 1 51B3FCC6
-P 5000 5600
-F 0 "R2" V 5080 5600 40  0000 C CNN
-F 1 "10k" V 5007 5601 40  0000 C CNN
-F 2 "Resistors_SMD:R_0805_HandSoldering" V 4930 5600 30  0001 C CNN
-F 3 "~" H 5000 5600 30  0000 C CNN
-	1    5000 5600
+P 5000 5750
+F 0 "R2" V 5080 5750 40  0000 C CNN
+F 1 "10k" V 5007 5751 40  0000 C CNN
+F 2 "Resistors_SMD:R_0805_HandSoldering" V 4930 5750 30  0001 C CNN
+F 3 "~" H 5000 5750 30  0000 C CNN
+	1    5000 5750
 	1    0    0    -1
 $EndComp
@@
 P 6900 4850
 F 0 "R4" V 6980 4850 40  0000 C CNN
-F 1 "1.123MEG" V 6907 4851 40  0000 C CNN
+F 1 "1.5MEG" V 6907 4851 40  0000 C CNN
 F 2 "Resistors_SMD:R_1206_HandSoldering" V 6830 4850 30  0001 C CNN
 F 3 "~" H 6900 4850 30  0000 C CNN
@@
 P 6000 2050
 F 0 "L1" V 5950 2050 40  0000 C CNN
-F 1 "150u" V 6100 2050 40  0000 C CNN
+F 1 "100u" V 6100 2050 40  0000 C CNN
 F 2 "Nixie:SRU1048-151Y" V 5850 2050 60  0000 C CNN
 F 3 "~" H 6000 2050 60  0000 C CNN
@@
 $EndComp
 Text HLabel 1200 4700 0    60   Input ~ 0
-180V_SHDN
+180V_EN
 $Comp
 L C-RESCUE-nixie_clock C7
@@
 Text Notes 8350 4000 0    60   ~ 0
 1in high caps\nONLY INSTALL TWO OF THESE!
-$Comp
-L +170V #PWR018
-U 1 1 57CCC588
-P 7650 2200
-F 0 "#PWR018" H 7650 2050 60  0001 C CNN
-F 1 "+170V" H 7650 2340 60  0000 C CNN
-F 2 "" H 7650 2200 60  0000 C CNN
-F 3 "" H 7650 2200 60  0000 C CNN
-	1    7650 2200
-	1    0    0    -1
-$EndComp
 Text Notes 6850 3050 0    60   ~ 0
 ES2F
-Wire Wire Line
-	6000 2350 6000 3600
-Wire Wire Line
-	6000 2750 6800 2750
-Connection ~ 6000 2750
-Wire Wire Line
-	7100 2750 9600 2750
-Wire Wire Line
-	8100 2950 8100 2750
-Connection ~ 8100 2750
-Wire Wire Line
-	8450 2950 8450 2750
-Connection ~ 8450 2750
-Wire Wire Line
-	8850 2950 8850 2750
-Connection ~ 8850 2750
-Wire Wire Line
-	9250 2950 9250 2750
-Connection ~ 9250 2750
-Wire Wire Line
-	8100 3350 8100 3550
-Wire Wire Line
-	8100 3550 9250 3550
-Wire Wire Line
-	9250 3550 9250 3350
-Wire Wire Line
-	8450 3350 8450 3550
-Connection ~ 8450 3550
-Wire Wire Line
-	8850 3350 8850 3550
-Connection ~ 8850 3550
-Wire Wire Line
-	8650 3550 8650 3700
-Connection ~ 8650 3550
-Wire Wire Line
-	6000 1500 6000 1750
-Wire Wire Line
-	4400 4300 5150 4300
-Wire Wire Line
-	5150 4300 5150 3800
-Wire Wire Line
-	5150 3800 5700 3800
-Wire Wire Line
-	6000 4000 6000 5350
-Wire Wire Line
-	4400 4500 6000 4500
-Connection ~ 6000 4500
-Wire Wire Line
-	4400 4850 6650 4850
-Wire Wire Line
-	6450 4850 6450 5150
-Wire Wire Line
-	6450 5150 6700 5150
-Connection ~ 6450 4850
-Wire Wire Line
-	7100 5150 7400 5150
-Wire Wire Line
-	7400 5150 7400 4850
-Wire Wire Line
-	7650 4850 7150 4850
-Wire Wire Line
-	7650 2200 7650 4850
-Connection ~ 7650 2750
-Connection ~ 7400 4850
-Wire Wire Line
-	5000 5350 5000 4850
-Connection ~ 5000 4850
-Wire Wire Line
-	3550 5350 3550 6050
-Wire Wire Line
-	3550 6050 6000 6050
-Wire Wire Line
-	5000 6050 5000 5850
-Wire Wire Line
-	3850 5350 3850 6050
-Connection ~ 3850 6050
-Wire Wire Line
-	3700 6050 3700 6200
-Connection ~ 3700 6050
-Wire Wire Line
-	6000 6050 6000 5850
-Connection ~ 5000 6050
-Wire Wire Line
-	3700 2750 3700 3650
-Wire Wire Line
-	4150 2950 4150 2850
-Wire Wire Line
-	3700 2850 4450 2850
-Connection ~ 3700 2850
-Wire Wire Line
-	4450 2850 4450 2950
-Connection ~ 4150 2850
-Wire Wire Line
-	4150 3350 4150 3450
-Wire Wire Line
-	4150 3450 4450 3450
-Wire Wire Line
-	4450 3450 4450 3350
-Wire Wire Line
-	4300 3450 4300 3550
-Connection ~ 4300 3450
-Wire Wire Line
-	2250 4150 2250 4500
-Wire Wire Line
-	2250 3500 2250 3650
-Wire Wire Line
-	2750 4600 2750 4500
-Wire Wire Line
-	2750 5000 2750 5150
-Wire Wire Line
-	10550 2100 10550 2150
-Wire Wire Line
-	10550 2950 10550 3050
-$Comp
-L MPSA42 Q?
-U 1 1 57FDD1C5
-P 10450 2750
-F 0 "Q?" H 10650 2825 50  0000 L CNN
-F 1 "MPSA42" H 10650 2750 50  0000 L CNN
-F 2 "TO-92" H 10650 2675 50  0000 L CIN
-F 3 "" H 10450 2750 50  0000 L CNN
-	1    10450 2750
-	1    0    0    -1
-$EndComp
-Wire Wire Line
-	10550 1600 10550 1500
 $Comp
 L +12V #PWR?
@@
 	0    1    1    0
 $EndComp
-Wire Wire Line
-	10100 2750 10250 2750
-$Comp
-L MPSA42 Q?
-U 1 1 57FDE608
-P 2150 4700
-F 0 "Q?" H 2350 4775 50  0000 L CNN
-F 1 "MPSA42" H 2350 4700 50  0000 L CNN
-F 2 "TO-92" H 2350 4625 50  0000 L CIN
-F 3 "" H 2150 4700 50  0000 L CNN
-	1    2150 4700
-	1    0    0    -1
-$EndComp
-Wire Wire Line
-	2250 4900 2250 5200
 $Comp
 L GND #PWR?
@@
 	0    1    1    0
 $EndComp
-Wire Wire Line
-	1850 4700 1950 4700
 $Comp
 L +12V #PWR?
@@
 	1    0    0    -1
 $EndComp
+$Comp
+L +180V #PWR?
+U 1 1 5820B873
+P 7650 2200
+F 0 "#PWR?" H 7650 2050 60  0001 C CNN
+F 1 "+180V" H 7650 2340 60  0000 C CNN
+F 2 "" H 7650 2200 60  0000 C CNN
+F 3 "" H 7650 2200 60  0000 C CNN
+	1    7650 2200
+	1    0    0    -1
+$EndComp
+$Comp
+L RVAR R?
+U 1 1 5820F775
+P 5000 5200
+F 0 "R?" V 5080 5150 50  0000 C CNN
+F 1 "5K" V 4920 5260 50  0000 C CNN
+F 2 "" H 5000 5200 50  0000 C CNN
+F 3 "" H 5000 5200 50  0000 C CNN
+	1    5000 5200
+	1    0    0    -1
+$EndComp
+Text Notes 6250 2500 1    60   ~ 0
+>2A max current
+$Comp
+L C-RESCUE-nixie_clock C?
+U 1 1 5821057A
+P 6550 1850
+F 0 "C?" H 6550 1950 40  0000 L CNN
+F 1 "100uF" H 6556 1765 40  0000 L CNN
+F 2 "Capacitors_Tantalum_SMD:TantalC_SizeD_EIA-7343_HandSoldering" H 6588 1700 30  0001 C CNN
+F 3 "~" H 6550 1850 60  0000 C CNN
+F 4 "35V" H 6650 1650 60  0000 C CNN "Voltage"
+	1    6550 1850
+	1    0    0    -1
+$EndComp
+Wire Wire Line
+	6000 2350 6000 3600
+Wire Wire Line
+	6000 2750 6800 2750
+Connection ~ 6000 2750
+Wire Wire Line
+	7100 2750 9600 2750
+Wire Wire Line
+	8100 2950 8100 2750
+Connection ~ 8100 2750
+Wire Wire Line
+	8450 2950 8450 2750
+Connection ~ 8450 2750
+Wire Wire Line
+	8850 2950 8850 2750
+Connection ~ 8850 2750
+Wire Wire Line
+	9250 2950 9250 2750
+Connection ~ 9250 2750
+Wire Wire Line
+	8100 3350 8100 3550
+Wire Wire Line
+	8100 3550 9250 3550
+Wire Wire Line
+	9250 3550 9250 3350
+Wire Wire Line
+	8450 3350 8450 3550
+Connection ~ 8450 3550
+Wire Wire Line
+	8850 3350 8850 3550
+Connection ~ 8850 3550
+Wire Wire Line
+	8650 3550 8650 3700
+Connection ~ 8650 3550
+Wire Wire Line
+	6000 1500 6000 1750
+Wire Wire Line
+	4400 4300 5150 4300
+Wire Wire Line
+	5150 4300 5150 3800
+Wire Wire Line
+	5150 3800 5700 3800
+Wire Wire Line
+	6000 4000 6000 5350
+Wire Wire Line
+	4400 4500 6000 4500
+Connection ~ 6000 4500
+Wire Wire Line
+	4400 4850 6650 4850
+Wire Wire Line
+	6450 4850 6450 5150
+Wire Wire Line
+	6450 5150 6700 5150
+Connection ~ 6450 4850
+Wire Wire Line
+	7100 5150 7400 5150
+Wire Wire Line
+	7400 5150 7400 4850
+Wire Wire Line
+	7650 4850 7150 4850
+Wire Wire Line
+	7650 2200 7650 4850
+Connection ~ 7650 2750
+Connection ~ 7400 4850
+Connection ~ 5000 4850
+Wire Wire Line
+	3550 5350 3550 6050
+Wire Wire Line
+	3550 6050 6000 6050
+Wire Wire Line
+	5000 6050 5000 6000
+Wire Wire Line
+	3850 5350 3850 6050
+Connection ~ 3850 6050
+Wire Wire Line
+	3700 6050 3700 6200
+Connection ~ 3700 6050
+Wire Wire Line
+	6000 6050 6000 5850
+Connection ~ 5000 6050
+Wire Wire Line
+	3700 2750 3700 3650
+Wire Wire Line
+	4150 2950 4150 2850
+Wire Wire Line
+	3700 2850 4450 2850
+Connection ~ 3700 2850
+Wire Wire Line
+	4450 2850 4450 2950
+Connection ~ 4150 2850
+Wire Wire Line
+	4150 3350 4150 3450
+Wire Wire Line
+	4150 3450 4450 3450
+Wire Wire Line
+	4450 3450 4450 3350
+Wire Wire Line
+	4300 3450 4300 3550
+Connection ~ 4300 3450
+Wire Wire Line
+	2250 4150 2250 4500
+Wire Wire Line
+	2250 3500 2250 3650
+Wire Wire Line
+	2750 4600 2750 4500
+Wire Wire Line
+	2750 5000 2750 5150
+Wire Wire Line
+	10550 2100 10550 2150
+Wire Wire Line
+	10550 2950 10550 3050
+Wire Wire Line
+	10550 1600 10550 1500
+Wire Wire Line
+	10100 2750 10250 2750
+Wire Wire Line
+	2250 4900 2250 5200
+Wire Wire Line
+	1850 4700 1950 4700
 Connection ~ 2250 4300
 Wire Wire Line
@@
 Wire Wire Line
 	3000 4300 2250 4300
+Wire Wire Line
+	5000 5450 5000 5500
+Wire Wire Line
+	5000 4950 5000 4850
+Wire Wire Line
+	6000 1600 6550 1600
+Wire Wire Line
+	6550 1600 6550 1650
+Connection ~ 6000 1600
+Wire Wire Line
+	6550 2050 6550 2150
+$Comp
+L GND #PWR?
+U 1 1 58210772
+P 6550 2150
+F 0 "#PWR?" H 6550 2150 30  0001 C CNN
+F 1 "GND" H 6550 2080 30  0001 C CNN
+F 2 "" H 6550 2150 60  0000 C CNN
+F 3 "" H 6550 2150 60  0000 C CNN
+	1    6550 2150
+	1    0    0    -1
+$EndComp
+Text Notes 6250 6000 1    60   ~ 0
+>2A max current
+$Comp
+L MMBTA42 Q?
+U 1 1 581FB66E
+P 10450 2750
+F 0 "Q?" H 10650 2825 50  0000 L CNN
+F 1 "MMBTA42" H 10650 2750 50  0000 L CNN
+F 2 "TO_SOT_Packages_SMD:SOT-23_Handsoldering" H 10650 2675 50  0001 L CIN
+F 3 "" H 10450 2750 50  0000 L CNN
+	1    10450 2750
+	1    0    0    -1
+$EndComp
+$Comp
+L MMBTA42 Q?
+U 1 1 581FB951
+P 2150 4700
+F 0 "Q?" H 2350 4775 50  0000 L CNN
+F 1 "MMBTA42" H 2350 4700 50  0000 L CNN
+F 2 "TO_SOT_Packages_SMD:SOT-23_Handsoldering" H 2350 4625 50  0001 L CIN
+F 3 "" H 2150 4700 50  0000 L CNN
+	1    2150 4700
+	1    0    0    -1
+$EndComp
 $EndSCHEMATC

Commit message: Updates to BOM
Start to update BOM for 180V supply
Parts:
- removed C7, C8: 47uF, Capacitors_ThroughHole:C_Radial_D12.5_L25_P5, symbol C-RESCUE-nixie_clock
- removed R?: 5K, symbol RVAR
- added R16: RVAR-TRIM, Nixie:67ZR5KLF, symbol RVAR-TRIM
- C2: value 68uF -> 10uF; footprint Capacitors_Tantalum_SMD:TantalC_SizeD_EIA-7343_HandSoldering -> Capacitors_SMD:C_1210_HandSoldering
- C20: renamed from C?; footprint Capacitors_Tantalum_SMD:TantalC_SizeD_EIA-7343_HandSoldering -> Capacitors_SMD:c_elec_6.3x7.7; Voltage 35V -> 25V
- L1: footprint Nixie:SRU1048-151Y -> Nixie:B82479A1104M
- U1: footprint Power_Integrations:PDIP-8 -> SMD_Packages:SOIC-8-N
- gave numbers to parts that had none: 4
Connections:
- wire segments 58 -> 54
- no-connect marks 0 -> 1
Other:
- note added: "1in high caps\nONLY INSTALL ONE OF THESE!"
- note removed: "1in high caps\nONLY INSTALL TWO OF THESE!"
Changed lines of the file:
@@
-$EndComp
-$Comp
-L C-RESCUE-nixie_clock C8
-U 1 1 51B3FCF0
-P 9250 3150
-F 0 "C8" H 9250 3250 40  0000 L CNN
-F 1 "47uF" H 9256 3065 40  0000 L CNN
-F 2 "Capacitors_ThroughHole:C_Radial_D12.5_L25_P5" H 9288 3000 30  0001 C CNN
-F 3 "~" H 9250 3150 60  0000 C CNN
-	1    9250 3150
-	1    0    0    -1
 $EndComp
 $Comp
@@
 F 0 "L1" V 5950 2050 40  0000 C CNN
 F 1 "100u" V 6100 2050 40  0000 C CNN
-F 2 "Nixie:SRU1048-151Y" V 5850 2050 60  0000 C CNN
+F 2 "Nixie:B82479A1104M" V 5850 2050 60  0000 C CNN
 F 3 "~" H 6000 2050 60  0000 C CNN
 	1    6000 2050
@@
 $EndComp
 $Comp
-L GND #PWR08
+L GND #PWR010
 U 1 1 51B3FD08
-P 8650 3700
-F 0 "#PWR08" H 8650 3700 30  0001 C CNN
-F 1 "GND" H 8650 3630 30  0001 C CNN
-F 2 "" H 8650 3700 60  0000 C CNN
-F 3 "" H 8650 3700 60  0000 C CNN
-	1    8650 3700
-	1    0    0    -1
-$EndComp
-$Comp
-L GND #PWR09
-U 1 1 51B3FD0E
-P 8650 3700
-F 0 "#PWR09" H 8650 3700 30  0001 C CNN
-F 1 "GND" H 8650 3630 30  0001 C CNN
-F 2 "" H 8650 3700 60  0000 C CNN
-F 3 "" H 8650 3700 60  0000 C CNN
-	1    8650 3700
-	1    0    0    -1
-$EndComp
-$Comp
-L GND #PWR010
+P 8300 3700
+F 0 "#PWR010" H 8300 3700 30  0001 C CNN
+F 1 "GND" H 8300 3630 30  0001 C CNN
+F 2 "" H 8300 3700 60  0000 C CNN
+F 3 "" H 8300 3700 60  0000 C CNN
+	1    8300 3700
+	1    0    0    -1
+$EndComp
+$Comp
+L GND #PWR011
 U 1 1 51B3FD20
 P 3700 6200
-F 0 "#PWR010" H 3700 6200 30  0001 C CNN
+F 0 "#PWR011" H 3700 6200 30  0001 C CNN
 F 1 "GND" H 3700 6130 30  0001 C CNN
 F 2 "" H 3700 6200 60  0000 C CNN
@@
 F 0 "U1" H 4050 3100 60  0000 C CNN
 F 1 "MAX1771" H 4050 3000 60  0000 C CNN
-F 2 "Power_Integrations:PDIP-8" H 3050 2900 60  0000 C CNN
+F 2 "SMD_Packages:SOIC-8-N" H 3050 2900 60  0000 C CNN
 F 3 "" H 4050 3100 60  0000 C CNN
 	1    3700 3400
@@
 P 4150 3150
 F 0 "C2" H 4150 3250 40  0000 L CNN
-F 1 "68uF" H 4156 3065 40  0000 L CNN
-F 2 "Capacitors_Tantalum_SMD:TantalC_SizeD_EIA-7343_HandSoldering" H 4188 3000 30  0001 C CNN
+F 1 "10uF" H 4156 3065 40  0000 L CNN
+F 2 "Capacitors_SMD:C_1210_HandSoldering" H 4188 3000 30  0001 C CNN
 F 3 "~" H 4150 3150 60  0000 C CNN
 	1    4150 3150
@@
 $EndComp
 $Comp
-L GND #PWR011
+L GND #PWR012
 U 1 1 51B3FD74
 P 4300 3550
-F 0 "#PWR011" H 4300 3550 30  0001 C CNN
+F 0 "#PWR012" H 4300 3550 30  0001 C CNN
 F 1 "GND" H 4300 3480 30  0001 C CNN
 F 2 "" H 4300 3550 60  0000 C CNN
@@
 $EndComp
 $Comp
-L GND #PWR012
+L GND #PWR013
 U 1 1 51B3FD8B
 P 2750 5150
-F 0 "#PWR012" H 2750 5150 30  0001 C CNN
+F 0 "#PWR013" H 2750 5150 30  0001 C CNN
 F 1 "GND" H 2750 5080 30  0001 C CNN
 F 2 "" H 2750 5150 60  0000 C CNN
@@
 $EndComp
 $Comp
-L GND #PWR013
+L GND #PWR014
 U 1 1 51B3FD9D
 P 10550 3050
-F 0 "#PWR013" H 10550 3050 30  0001 C CNN
+F 0 "#PWR014" H 10550 3050 30  0001 C CNN
 F 1 "GND" H 10550 2980 30  0001 C CNN
 F 2 "" H 10550 3050 60  0000 C CNN
@@
 Text HLabel 1200 4700 0    60   Input ~ 0
 180V_EN
-$Comp
-L C-RESCUE-nixie_clock C7
-U 1 1 575BD4EC
-P 8850 3150
-F 0 "C7" H 8850 3250 40  0000 L CNN
-F 1 "47uF" H 8856 3065 40  0000 L CNN
-F 2 "Capacitors_ThroughHole:C_Radial_D12.5_L25_P5" H 8888 3000 30  0001 C CNN
-F 3 "~" H 8850 3150 60  0000 C CNN
-	1    8850 3150
-	1    0    0    -1
-$EndComp
-$Comp
-L C-RESCUE-nixie_clock C6
-U 1 1 575BD540
-P 8450 3150
-F 0 "C6" H 8450 3250 40  0000 L CNN
-F 1 "47uF" H 8456 3065 40  0000 L CNN
-F 2 "Capacitors_ThroughHole:C_Radial_D12.5_L25_P5" H 8488 3000 30  0001 C CNN
-F 3 "~" H 8450 3150 60  0000 C CNN
-	1    8450 3150
-	1    0    0    -1
-$EndComp
-$Comp
-L C-RESCUE-nixie_clock C5
-U 1 1 575BD5B4
-P 8100 3150
-F 0 "C5" H 8100 3250 40  0000 L CNN
-F 1 "47uF" H 8106 3065 40  0000 L CNN
-F 2 "Capacitors_ThroughHole:C_Radial_D12.5_L25_P5" H 8138 3000 30  0001 C CNN
-F 3 "~" H 8100 3150 60  0000 C CNN
-	1    8100 3150
-	1    0    0    -1
-$EndComp
 $Comp
 L IPB50R199CP Q1
@@
 $EndComp
 $Comp
-L +12V #PWR014
+L +12V #PWR015
 U 1 1 575E707A
 P 3700 2750
-F 0 "#PWR014" H 3700 2600 50  0001 C CNN
+F 0 "#PWR015" H 3700 2600 50  0001 C CNN
 F 1 "+12V" H 3700 2890 50  0000 C CNN
 F 2 "" H 3700 2750 50  0000 C CNN
@@
 $EndComp
 $Comp
-L +12V #PWR015
+L +12V #PWR016
 U 1 1 575E7381
 P 6000 1500
-F 0 "#PWR015" H 6000 1350 50  0001 C CNN
+F 0 "#PWR016" H 6000 1350 50  0001 C CNN
 F 1 "+12V" H 6000 1640 50  0000 C CNN
 F 2 "" H 6000 1500 50  0000 C CNN
@@
 $EndComp
 $Comp
-L PWR_FLAG #FLG016
+L PWR_FLAG #FLG017
 U 1 1 57671EA9
 P 8100 2750
-F 0 "#FLG016" H 8100 2845 50  0001 C CNN
+F 0 "#FLG017" H 8100 2845 50  0001 C CNN
 F 1 "PWR_FLAG" H 8100 2930 50  0000 C CNN
 F 2 "" H 8100 2750 50  0000 C CNN
@@
 	1    0    0    -1
 $EndComp
-Text Notes 8350 4000 0    60   ~ 0
-1in high caps\nONLY INSTALL TWO OF THESE!
+Text Notes 8000 4000 0    60   ~ 0
+1in high caps\nONLY INSTALL ONE OF THESE!
 Text Notes 6850 3050 0    60   ~ 0
 ES2F
 $Comp
-L +12V #PWR?
+L +12V #PWR018
 U 1 1 57FDD331
 P 10550 1500
-F 0 "#PWR?" H 10550 1350 50  0001 C CNN
+F 0 "#PWR018" H 10550 1350 50  0001 C CNN
 F 1 "+12V" H 10550 1640 50  0000 C CNN
 F 2 "" H 10550 1500 50  0000 C CNN
@@
 $EndComp
 $Comp
-L R-RESCUE-nixie_clock R?
+L R-RESCUE-nixie_clock R17
 U 1 1 57FDD39C
 P 9850 2750
-F 0 "R?" V 9930 2750 40  0000 C CNN
+F 0 "R17" V 9930 2750 40  0000 C CNN
 F 1 "470k" V 9857 2751 40  0000 C CNN
 F 2 "Resistors_SMD:R_0805_HandSoldering" V 9780 2750 30  0001 C CNN
@@
 $EndComp
 $Comp
-L GND #PWR?
+L GND #PWR019
 U 1 1 57FDE875
 P 2250 5200
-F 0 "#PWR?" H 2250 5200 30  0001 C CNN
+F 0 "#PWR019" H 2250 5200 30  0001 C CNN
 F 1 "GND" H 2250 5130 30  0001 C CNN
 F 2 "" H 2250 5200 60  0000 C CNN
@@
 $EndComp
 $Comp
-L R-RESCUE-nixie_clock R?
+L R-RESCUE-nixie_clock R15
 U 1 1 57FDE8BF
 P 1600 4700
-F 0 "R?" V 1680 4700 40  0000 C CNN
+F 0 "R15" V 1680 4700 40  0000 C CNN
 F 1 "4.7k" V 1607 4701 40  0000 C CNN
 F 2 "Resistors_SMD:R_0805_HandSoldering" V 1530 4700 30  0001 C CNN
@@
 $EndComp
 $Comp
-L +12V #PWR?
+L +12V #PWR020
 U 1 1 57FDE9DA
 P 2250 3500
-F 0 "#PWR?" H 2250 3350 50  0001 C CNN
+F 0 "#PWR020" H 2250 3350 50  0001 C CNN
 F 1 "+12V" H 2250 3640 50  0000 C CNN
 F 2 "" H 2250 3500 50  0000 C CNN
@@
 $EndComp
 $Comp
-L +180V #PWR?
+L +180V #PWR021
 U 1 1 5820B873
 P 7650 2200
-F 0 "#PWR?" H 7650 2050 60  0001 C CNN
+F 0 "#PWR021" H 7650 2050 60  0001 C CNN
 F 1 "+180V" H 7650 2340 60  0000 C CNN
 F 2 "" H 7650 2200 60  0000 C CNN
@@
 	1    0    0    -1
 $EndComp
-$Comp
-L RVAR R?
-U 1 1 5820F775
-P 5000 5200
-F 0 "R?" V 5080 5150 50  0000 C CNN
-F 1 "5K" V 4920 5260 50  0000 C CNN
-F 2 "" H 5000 5200 50  0000 C CNN
-F 3 "" H 5000 5200 50  0000 C CNN
-	1    5000 5200
-	1    0    0    -1
-$EndComp
 Text Notes 6250 2500 1    60   ~ 0
 >2A max current
 $Comp
-L C-RESCUE-nixie_clock C?
+L C-RESCUE-nixie_clock C20
 U 1 1 5821057A
 P 6550 1850
-F 0 "C?" H 6550 1950 40  0000 L CNN
+F 0 "C20" H 6550 1950 40  0000 L CNN
 F 1 "100uF" H 6556 1765 40  0000 L CNN
-F 2 "Capacitors_Tantalum_SMD:TantalC_SizeD_EIA-7343_HandSoldering" H 6588 1700 30  0001 C CNN
+F 2 "Capacitors_SMD:c_elec_6.3x7.7" H 6588 1700 30  0001 C CNN
 F 3 "~" H 6550 1850 60  0000 C CNN
-F 4 "35V" H 6650 1650 60  0000 C CNN "Voltage"
+F 4 "25V" H 6650 1650 60  0000 C CNN "Voltage"
 	1    6550 1850
 	1    0    0    -1
@@
 Connection ~ 8450 2750
 Wire Wire Line
-	8850 2950 8850 2750
-Connection ~ 8850 2750
-Wire Wire Line
-	9250 2950 9250 2750
-Connection ~ 9250 2750
-Wire Wire Line
 	8100 3350 8100 3550
-Wire Wire Line
-	8100 3550 9250 3550
-Wire Wire Line
-	9250 3550 9250 3350
-Wire Wire Line
-	8450 3350 8450 3550
-Connection ~ 8450 3550
-Wire Wire Line
-	8850 3350 8850 3550
-Connection ~ 8850 3550
-Wire Wire Line
-	8650 3550 8650 3700
-Connection ~ 8650 3550
 Wire Wire Line
 	6000 1500 6000 1750
@@
 	6550 2050 6550 2150
 $Comp
-L GND #PWR?
+L GND #PWR022
 U 1 1 58210772
 P 6550 2150
-F 0 "#PWR?" H 6550 2150 30  0001 C CNN
+F 0 "#PWR022" H 6550 2150 30  0001 C CNN
 F 1 "GND" H 6550 2080 30  0001 C CNN
 F 2 "" H 6550 2150 60  0000 C CNN
@@
 >2A max current
 $Comp
-L MMBTA42 Q?
+L MMBTA42 Q3
 U 1 1 581FB66E
 P 10450 2750
-F 0 "Q?" H 10650 2825 50  0000 L CNN
+F 0 "Q3" H 10650 2825 50  0000 L CNN
 F 1 "MMBTA42" H 10650 2750 50  0000 L CNN
 F 2 "TO_SOT_Packages_SMD:SOT-23_Handsoldering" H 10650 2675 50  0001 L CIN
@@
 $EndComp
 $Comp
-L MMBTA42 Q?
+L MMBTA42 Q2
 U 1 1 581FB951
 P 2150 4700
-F 0 "Q?" H 2350 4775 50  0000 L CNN
+F 0 "Q2" H 2350 4775 50  0000 L CNN
 F 1 "MMBTA42" H 2350 4700 50  0000 L CNN
 F 2 "TO_SOT_Packages_SMD:SOT-23_Handsoldering" H 2350 4625 50  0001 L CIN
@@
 	1    0    0    -1
 $EndComp
+$Comp
+L C-RESCUE-nixie_clock C6
+U 1 1 575BD540
+P 8450 3150
+F 0 "C6" H 8450 3250 40  0000 L CNN
+F 1 "47uF" H 8456 3065 40  0000 L CNN
+F 2 "Capacitors_ThroughHole:C_Radial_D12.5_L25_P5" H 8488 3000 30  0001 C CNN
+F 3 "~" H 8450 3150 60  0000 C CNN
+	1    8450 3150
+	1    0    0    -1
+$EndComp
+$Comp
+L C-RESCUE-nixie_clock C5
+U 1 1 575BD5B4
+P 8100 3150
+F 0 "C5" H 8100 3250 40  0000 L CNN
+F 1 "47uF" H 8106 3065 40  0000 L CNN
+F 2 "Capacitors_ThroughHole:C_Radial_D12.5_L25_P5" H 8138 3000 30  0001 C CNN
+F 3 "~" H 8100 3150 60  0000 C CNN
+	1    8100 3150
+	1    0    0    -1
+$EndComp
+Wire Wire Line
+	8450 3350 8450 3550
+Wire Wire Line
+	8450 3550 8100 3550
+Wire Wire Line
+	8300 3700 8300 3550
+Connection ~ 8300 3550
+$Comp
+L RVAR-TRIM R16
+U 1 1 58215A71
+P 5000 5200
+F 0 "R16" V 5080 5150 50  0000 C CNN
+F 1 "RVAR-TRIM" V 4850 5200 50  0000 C CNN
+F 2 "Nixie:67ZR5KLF" V 4750 5200 50  0000 C CNN
+F 3 "" H 5000 5200 50  0000 C CNN
+	1    5000 5200
+	1    0    0    -1
+$EndComp
+NoConn ~ 5200 5200
 $EndSCHEMATC
