File: hw/kicad_v1_1/projects/tube_shield/colon_tubes.sch (KiCad schematic (older format))
At the start: 8 parts, among them Q10 MPSA42, Q11 MPSA42

Commit message: Update
Begin work on updating for rev1.1.
Parts:
- removed Q10, Q11: MPSA42, TO_SOT_Packages_SMD:SOT-23_Handsoldering, symbol MPSA42
- added Q1, Q2: MMBTA42, TO_SOT_Packages_SMD:SOT-23_Handsoldering, symbol MMBTA42
- R30, R31: value 24k -> 100k
Connections:
- net GND: now also Q1.2 (E), Q2.2 (E)
- net at N1.2: now also Q2.3 (C)
- net at N2.2: now also Q1.3 (C)
- net at R32.1: now also Q1.1 (B)
- net at R33.1: now also Q2.1 (B)
Changed lines of the file:
@@
 SEL_COL
-$Comp
-L MPSA42 Q10
-U 1 1 575FD4F2
-P 6350 4200
-F 0 "Q10" H 6550 4275 50  0000 L CNN
-F 1 "MPSA42" H 6550 4200 50  0000 L CNN
-F 2 "TO_SOT_Packages_SMD:SOT-23_Handsoldering" H 6550 4125 50  0001 L CIN
-F 3 "" H 6350 4200 50  0000 L CNN
-	1    6350 4200
-	1    0    0    -1
-$EndComp
-$Comp
-L MPSA42 Q11
-U 1 1 575FD574
-P 7500 4200
-F 0 "Q11" H 7700 4275 50  0000 L CNN
-F 1 "MPSA42" H 7700 4200 50  0000 L CNN
-F 2 "TO_SOT_Packages_SMD:SOT-23_Handsoldering" H 7700 4125 50  0001 L CIN
-F 3 "" H 7500 4200 50  0000 L CNN
-	1    7500 4200
-	1    0    0    -1
-$EndComp
 $Comp
 L R R30
@@
 P 4550 2800
 F 0 "R30" V 4630 2800 50  0000 C CNN
-F 1 "24k" V 4550 2800 50  0000 C CNN
+F 1 "100k" V 4550 2800 50  0000 C CNN
 F 2 "Resistors_SMD:R_0805_HandSoldering" V 4480 2800 50  0001 C CNN
 F 3 "" H 4550 2800 50  0000 C CNN
@@
 P 4550 3650
 F 0 "R31" V 4630 3650 50  0000 C CNN
-F 1 "24k" V 4550 3650 50  0000 C CNN
+F 1 "100k" V 4550 3650 50  0000 C CNN
 F 2 "Resistors_SMD:R_0805_HandSoldering" V 4480 3650 50  0001 C CNN
 F 3 "" H 4550 3650 50  0000 C CNN
@@
 	1    0    0    -1
 $EndComp
+$Comp
+L MMBTA42 Q1
+U 1 1 581EED90
+P 6350 4200
+F 0 "Q1" H 6550 4275 50  0000 L CNN
+F 1 "MMBTA42" H 6550 4200 50  0000 L CNN
+F 2 "TO_SOT_Packages_SMD:SOT-23_Handsoldering" H 6550 4125 50  0001 L CIN
+F 3 "" H 6350 4200 50  0000 L CNN
+	1    6350 4200
+	1    0    0    -1
+$EndComp
+$Comp
+L MMBTA42 Q2
+U 1 1 581EEE1A
+P 7500 4200
+F 0 "Q2" H 7700 4275 50  0000 L CNN
+F 1 "MMBTA42" H 7700 4200 50  0000 L CNN
+F 2 "TO_SOT_Packages_SMD:SOT-23_Handsoldering" H 7700 4125 50  0001 L CIN
+F 3 "" H 7500 4200 50  0000 L CNN
+	1    7500 4200
+	1    0    0    -1
+$EndComp

Commit message: Complete with errors
Check in before moving header. Currently the headers don't match up. If
I'm going to connect them with standard header I need to move it
significantly. Check in as a roll back point.
Parts:
- R30, R31: footprint Resistors_SMD:R_0805_HandSoldering -> Resistors_SMD:R_1206_HandSoldering
Changed lines of the file:
@@
 F 0 "R30" V 4630 2800 50  0000 C CNN
 F 1 "100k" V 4550 2800 50  0000 C CNN
-F 2 "Resistors_SMD:R_0805_HandSoldering" V 4480 2800 50  0001 C CNN
+F 2 "Resistors_SMD:R_1206_HandSoldering" V 4480 2800 50  0001 C CNN
 F 3 "" H 4550 2800 50  0000 C CNN
 	1    4550 2800
-	0    1    1    0
-$EndComp
-$Comp
-L R R31
-U 1 1 575E0A55
-P 4550 3650
-F 0 "R31" V 4630 3650 50  0000 C CNN
-F 1 "100k" V 4550 3650 50  0000 C CNN
-F 2 "Resistors_SMD:R_0805_HandSoldering" V 4480 3650 50  0001 C CNN
-F 3 "" H 4550 3650 50  0000 C CNN
-	1    4550 3650
 	0    1    1    0
 $EndComp
@@
 	1    0    0    -1
 $EndComp
+$Comp
+L R R31
+U 1 1 575E0A55
+P 4550 3650
+F 0 "R31" V 4630 3650 50  0000 C CNN
+F 1 "100k" V 4550 3650 50  0000 C CNN
+F 2 "Resistors_SMD:R_1206_HandSoldering" V 4480 3650 50  0001 C CNN
+F 3 "" H 4550 3650 50  0000 C CNN
+	1    4550 3650
+	0    1    1    0
+$EndComp
 $EndSCHEMATC
