File: hw/kicad_v1_1/projects/tube_shield/nixie_tubes.sch (KiCad schematic (older format))
At the start: 8 parts

Commit message: Complete with errors
Check in before moving header. Currently the headers don't match up. If
I'm going to connect them with standard header I need to move it
significantly. Check in as a roll back point.
Parts:
- R1, R10, R2, R3: footprint Resistors_SMD:R_0805_HandSoldering -> Resistors_SMD:R_1206_HandSoldering
Changed lines of the file:
@@
 F 0 "R10" V 3580 1200 40  0000 C CNN
 F 1 "15k" V 3507 1201 40  0000 C CNN
-F 2 "Resistors_SMD:R_0805_HandSoldering" V 3430 1200 30  0001 C CNN
+F 2 "Resistors_SMD:R_1206_HandSoldering" V 3430 1200 30  0001 C CNN
 F 3 "~" H 3500 1200 30  0000 C CNN
 	1    3500 1200
@@
 F 0 "R2" V 7830 1150 40  0000 C CNN
 F 1 "15k" V 7757 1151 40  0000 C CNN
-F 2 "Resistors_SMD:R_0805_HandSoldering" V 7680 1150 30  0001 C CNN
+F 2 "Resistors_SMD:R_1206_HandSoldering" V 7680 1150 30  0001 C CNN
 F 3 "~" H 7750 1150 30  0000 C CNN
 	1    7750 1150
@@
 F 0 "R1" V 3530 3900 40  0000 C CNN
 F 1 "15k" V 3457 3901 40  0000 C CNN
-F 2 "Resistors_SMD:R_0805_HandSoldering" V 3380 3900 30  0001 C CNN
+F 2 "Resistors_SMD:R_1206_HandSoldering" V 3380 3900 30  0001 C CNN
 F 3 "~" H 3450 3900 30  0000 C CNN
 	1    3450 3900
@@
 F 0 "R3" V 7830 3900 40  0000 C CNN
 F 1 "12k" V 7757 3901 40  0000 C CNN
-F 2 "Resistors_SMD:R_0805_HandSoldering" V 7680 3900 30  0001 C CNN
+F 2 "Resistors_SMD:R_1206_HandSoldering" V 7680 3900 30  0001 C CNN
 F 3 "~" H 7750 3900 30  0000 C CNN
 	1    7750 3900
