File: hw/kicad_v1_1/projects/tube_shield/nixie_control.sch (KiCad schematic (older format))
At the start: 8 parts, among them U1 K155ID1, U2 K155ID1, U3 K155ID1, U4 K155ID1

Commit message: Final Release
Update with trimming and bug fixes. This is what is being delivered as a
V1.1.0 release.
Parts:
- C1, C2, C3, C4: footprint (none) -> Capacitors_SMD:C_0805_HandSoldering
Changed lines of the file:
@@
 F 0 "C2" H 1325 2950 50  0000 L CNN
 F 1 "0.1u" H 1325 2750 50  0000 L CNN
-F 2 "" H 1338 2700 50  0000 C CNN
+F 2 "Capacitors_SMD:C_0805_HandSoldering" H 1338 2700 50  0001 C CNN
 F 3 "" H 1300 2850 50  0000 C CNN
 	1    1300 2850
@@
 F 0 "C3" H 5875 2900 50  0000 L CNN
 F 1 "0.1u" H 5875 2700 50  0000 L CNN
-F 2 "" H 5888 2650 50  0000 C CNN
+F 2 "Capacitors_SMD:C_0805_HandSoldering" H 5888 2650 50  0001 C CNN
 F 3 "" H 5850 2800 50  0000 C CNN
 	1    5850 2800
@@
 F 0 "C1" H 1225 5250 50  0000 L CNN
 F 1 "0.1u" H 1225 5050 50  0000 L CNN
-F 2 "" H 1238 5000 50  0000 C CNN
+F 2 "Capacitors_SMD:C_0805_HandSoldering" H 1238 5000 50  0001 C CNN
 F 3 "" H 1200 5150 50  0000 C CNN
 	1    1200 5150
@@
 F 0 "C4" H 5875 5250 50  0000 L CNN
 F 1 "0.1u" H 5875 5050 50  0000 L CNN
-F 2 "" H 5888 5000 50  0000 C CNN
+F 2 "Capacitors_SMD:C_0805_HandSoldering" H 5888 5000 50  0001 C CNN
 F 3 "" H 5850 5150 50  0000 C CNN
 	1    5850 5150
